File: Reg-LT.sch (EAGLE design)
At the start: 64 parts, among them IC1 MEGA8-AI, IC2 DS1813-SMD, IC3 LM1117IMPX-3.3, IC4 LM321MF, IC5 LM321MF, Q1 20 MHz, X1 22-23-2021, X2 MKDSN1,5/3-5,08, X3 MKDSN1,5/3-5,08, X4 MKDSN1,5/3-5,08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

Commit message: sd-card no-module
Parts:
- removed U$2: SD-CARDSD-MODULE2X8-H, MyLib:SD-CARDSD-MODULE2X8-H
- added J1: ATTEND-MICROSD-112, MyLib:ATTEND-MICROSD-112
- added R20: 10k, rcl:R-EU_R0805
Connections:
- new net SD_DETECT: IC1.ADC6, J1.CD, R20.1
- net +3V3: now also J1.VDD, R20.2
- net +5V: no longer U$2.+5V
- net CS_SD: no longer U$2.CS
- net GND: now also J1.GND, J1.S@1, J1.S@2, J1.VSS(GND); no longer U$2.GND@1, U$2.GND@2
- net MISO: now also J1.DAT0(DO); no longer U$2.MISO
- net MOSI: now also J1.CMD(DI); no longer U$2.MOSI
- net SCK: now also J1.CLK(SCLK); no longer U$2.SCK

Commit message: timer - no-module
Parts:
- removed C15, C16: 0.1, rcl:C-EUC0805
- removed JP6: (no value), pinhead:PINHD-1X7
- removed LED1, LED2, LED3, LED4: (no value), led:LEDCHIP-LED0805
- removed R18, R19: 1k, rcl:R-EU_R0805
- removed U$3: RTCRTC_MODULE-1X6H, MyLib:RTCRTC_MODULE-1X6H
- removed U$4: LM7805TO-220-VERT, MyLib:LM7805TO-220-VERT
- added D3: BAT54S, diode:BAT54S
- added D4: 1N4004, diode:1N4004
- added G1: CR2032H, MyLib:CR2032H
- added IC7: PCF8583T, MyLib:PCF8583T
- added JP3: (no value), pinhead:PINHD-1X6
- added Q2: (no value), MyLib:MA306
- added X6: MKDSN1,5/3-5,08, con-phoenix-508:MKDSN1,5/3-5,08
- C5: value (none) -> 0.1; device rcl:CPOL-EU153CLV-0605 -> rcl:C-EUC0805
- R1, R17: value 1k -> 100
Connections:
- removed net +5V: C15.1, C16.1, C5.+, IC3.IN, JP6.2, U$3.VCC, U$4.VOUT
- removed net N$32: LED4.A, R19.1
- new net N$15: IC7.OSCI, Q2.1
- new net N$16: IC7.OSCO, Q2.2
- new net N$33: G1.+, IC7.A0
- net +3V3: now also C5.1, D3.C2, IC7.VDD, X6-3.KL
- net GND: now also C5.2, D3.A1, G1.-, IC7.VSS, JP3.1, R17.1, X6-1.KL; no longer C15.2, C16.2, C5.-, JP6.1, LED1.C, LED2.C, LED3.C, LED4.C, U$3.GND, U$4.GND
- net N$29: now also D3.C1A2, R1.2; no longer LED1.A, R1.1
- net N$30: now also R1.1, X6-2.KL; no longer LED2.A, R17.1
- net N$31: now also R17.2; no longer LED3.A, R18.1
- net PC1: now also JP3.2; no longer JP6.3
- net PC2: now also JP3.3; no longer JP6.4
- net PC3: now also JP3.4; no longer JP6.5
- net PW: now also IC3.IN; no longer U$4.VIN
- net RX_ESP: no longer R19.2
- net SCL: now also IC7.SCL, JP3.6; no longer JP6.7, R1.2, U$3.SCL
- net SDA: now also IC7.SDA, JP3.5; no longer JP6.6, R17.2, U$3.SDA
- net TX_ESP: no longer R18.2
Other:
- moved on the sheet: C14, R1, R17, X1-1, X1-2

Commit message: no amplifires
Parts:
- removed C17, C6: 10,0, rcl:C-EUC0805
- removed D3: BAT54S, diode:BAT54S
- removed D4: 1N4004, diode:1N4004
- removed IC4, IC5: LM321MF, linear:LM321MF
- removed R1, R17: 100, rcl:R-EU_R0805
- removed R13, R15: 10k, rcl:R-EU_R0805
- removed R14, R16: 10k, rcl:R-TRIMM3214W
- removed X2, X3: MKDSN1,5/3-5,08, con-phoenix-508:MKDSN1,5/3-5,08
- added D5, D6: 1N4148DO35-7, diode:1N4148DO35-7
- added X7: MKDSN1,5/2-5,08, con-phoenix-508:MKDSN1,5/2-5,08
- D1, D2: value BAT54S -> BAV199; device diode:BAT54S -> diode:BAV199
- R2, R9: value 100 -> (none); device rcl:R-EU_R0805 -> rcl:R-EU_VMTA55
- R3, R6: value 1.5k -> (none); device rcl:R-EU_R0805 -> rcl:R-EU_VMTA55
- X6: value MKDSN1,5/3-5,08 -> MKDSN1,5/2-5,08; device con-phoenix-508:MKDSN1,5/3-5,08 -> con-phoenix-508:MKDSN1,5/2-5,08
Connections:
- removed net N$13: D2.C1A2, R3.1, R9.2
- removed net N$17: IC5.-IN, R15.2, R16.S
- removed net N$29: D3.C1A2, R1.2
- removed net N$30: R1.1, X6-2.KL
- removed net N$31: R17.2
- removed net N$70: C6.1, IC4.+IN, R6.2
- removed net N$8: C17.1, IC5.+IN, R3.2
- removed net RESET_ESP: BTN2.1, R11.1, U$1.GPIO16, U$1.RESET
- net +3V3: now also D1.C, D2.C; no longer D1.C2, D2.C2, D3.C2, IC4.V+, IC5.V+, X2-3.KL, X3-3.KL, X6-3.KL
- net GND: now also D1.A, D2.A, R6.1, R9.1, X7-1.KL; no longer C17.2, C6.2, D1.A1, D2.A1, D3.A1, IC4.V-, IC5.V-, R13.1, R15.1, R17.1, X2-1.KL, X3-1.KL
- net N$1: now also D1.AC, D5.A; no longer D1.C1A2, R6.1
- net N$14: now also R2.1, X6-2.KL; no longer R9.1, X3-2.KL
- net N$24: now also D5.C, R6.2; no longer IC5.OUT, R16.E
- net N$5: now also R3.1, X7-2.KL; no longer R2.1, X2-2.KL
- net N$6: now also D2.AC, D6.A, R3.2; no longer IC4.-IN, R13.2, R14.S
- net N$7: now also D6.C, R9.2; no longer IC4.OUT, R14.E
- net T0: now also BTN2.1, R11.1, U$1.GPIO16, U$1.RESET
Other:
- moved on the sheet: R2, R3, R6, R9, X6-1, X6-2

Commit message: input-rectifier
Parts:
- removed D1, D2: BAV199, diode:BAV199
- removed D5, D6: 1N4148DO35-7, diode:1N4148DO35-7
- removed R2, R3: (no value), rcl:R-EU_VMTA55
- added B1, B2: DF08S, rectifier:DF08S
Connections:
- removed net N$14: R2.1, X6-2.KL
- removed net N$6: D2.AC, D6.A, R3.2
- new net N$13: B1.AC1, X6-2.KL
- new net N$8: B1.AC2, X6-1.KL
- net +3V3: no longer D1.C, D2.C
- net GND: now also B1.-, B2.-; no longer D1.A, D2.A, X6-1.KL, X7-1.KL
- net N$1: now also B2.AC1, X7-2.KL; no longer D1.AC, D5.A, R2.2
- net N$24: now also B1.+; no longer D5.C
- net N$5: now also B2.AC2, X7-1.KL; no longer R3.1, X7-2.KL
- net N$7: now also B2.+; no longer D6.C
Other:
- moved on the sheet: X6-1, X6-2, X7-1, X7-2
Changed lines of the file:
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@@
 <part name="JP3" library="pinhead" deviceset="PINHD-1X6" device=""/>
 <part name="C5" library="rcl" deviceset="C-EU" device="C0805" value="0.1"/>
-<part name="R2" library="rcl" deviceset="R-EU_" device="VMTA55"/>
-<part name="R3" library="rcl" deviceset="R-EU_" device="VMTA55"/>
-<part name="D1" library="diode" deviceset="BAV199" device=""/>
-<part name="D2" library="diode" deviceset="BAV199" device=""/>
-<part name="GND3" library="supply1" deviceset="GND" device=""/>
-<part name="GND6" library="supply1" deviceset="GND" device=""/>
-<part name="+3V2" library="supply1" deviceset="+3V3" device=""/>
-<part name="+3V5" library="supply1" deviceset="+3V3" device=""/>
-<part name="D5" library="diode" deviceset="1N4148" device="DO35-7"/>
-<part name="D6" library="diode" deviceset="1N4148" device="DO35-7"/>
 <part name="R6" library="rcl" deviceset="R-EU_" device="VMTA55"/>
 <part name="R9" library="rcl" deviceset="R-EU_" device="VMTA55"/>
@@
 <part name="X6" library="con-phoenix-508" deviceset="MKDSN1,5/2-5,08" device=""/>
 <part name="X7" library="con-phoenix-508" deviceset="MKDSN1,5/2-5,08" device=""/>
+<part name="B1" library="rectifier" deviceset="DF*S" device="" technology="08"/>
+<part name="B2" library="rectifier" deviceset="DF*S" device="" technology="08"/>
 </parts>
 <sheets>
@@
 <instance part="GND22" gate="1" x="-185.42" y="27.94"/>
 <instance part="C7" gate="G$1" x="-144.78" y="-55.88"/>
-<instance part="GND5" gate="1" x="-111.76" y="71.12"/>
+<instance part="GND5" gate="1" x="-121.92" y="68.58"/>
 <instance part="U$1" gate="G$1" x="63.5" y="35.56"/>
 <instance part="+3V3" gate="G$1" x="-116.84" y="53.34"/>
@@
 <instance part="C14" gate="G$1" x="-241.3" y="-60.96"/>
 <instance part="GND21" gate="1" x="-241.3" y="-68.58"/>
-<instance part="GND28" gate="1" x="-111.76" y="111.76"/>
+<instance part="GND28" gate="1" x="-121.92" y="109.22"/>
 <instance part="JP2" gate="A" x="63.5" y="93.98"/>
 <instance part="GND31" gate="1" x="81.28" y="-78.74"/>
@@
 <instance part="JP3" gate="A" x="104.14" y="-83.82"/>
 <instance part="C5" gate="G$1" x="-137.16" y="-55.88"/>
-<instance part="R2" gate="G$1" x="-104.14" y="121.92"/>
-<instance part="R3" gate="G$1" x="-104.14" y="81.28"/>
-<instance part="D1" gate="G$1" x="-96.52" y="121.92" rot="MR270"/>
-<instance part="D2" gate="G$1" x="-96.52" y="81.28" rot="MR270"/>
-<instance part="GND3" gate="1" x="-96.52" y="111.76"/>
-<instance part="GND6" gate="1" x="-96.52" y="71.12"/>
-<instance part="+3V2" gate="G$1" x="-96.52" y="132.08"/>
-<instance part="+3V5" gate="G$1" x="-96.52" y="91.44"/>
-<instance part="D5" gate="G$1" x="-83.82" y="121.92"/>
-<instance part="D6" gate="G$1" x="-83.82" y="81.28"/>
 <instance part="R6" gate="G$1" x="-78.74" y="116.84" rot="R90"/>
 <instance part="R9" gate="G$1" x="-78.74" y="76.2" rot="R90"/>
 <instance part="GND13" gate="1" x="-78.74" y="68.58"/>
 <instance part="GND23" gate="1" x="-78.74" y="109.22"/>
-<instance part="X6" gate="-1" x="-114.3" y="116.84" rot="R180"/>
-<instance part="X6" gate="-2" x="-114.3" y="121.92" rot="R180"/>
-<instance part="X7" gate="-1" x="-114.3" y="76.2" rot="R180"/>
-<instance part="X7" gate="-2" x="-114.3" y="81.28" rot="R180"/>
+<instance part="X6" gate="-1" x="-129.54" y="114.3" rot="R180"/>
+<instance part="X6" gate="-2" x="-129.54" y="129.54" rot="R180"/>
+<instance part="X7" gate="-1" x="-129.54" y="73.66" rot="R180"/>
+<instance part="X7" gate="-2" x="-129.54" y="88.9" rot="R180"/>
+<instance part="B1" gate="G$1" x="-114.3" y="121.92"/>
+<instance part="B2" gate="G$1" x="-114.3" y="81.28"/>
 </instances>
 <busses>
@@
 </segment>
 <segment>
-<pinref part="GND5" gate="1" pin="GND"/>
-<wire x1="-111.76" y1="73.66" x2="-111.76" y2="76.2" width="0.1524" layer="91"/>
-<pinref part="X7" gate="-1" pin="KL"/>
-</segment>
-<segment>
-<pinref part="GND28" gate="1" pin="GND"/>
-<wire x1="-111.76" y1="114.3" x2="-111.76" y2="116.84" width="0.1524" layer="91"/>
-<pinref part="X6" gate="-1" pin="KL"/>
-</segment>
-<segment>
 <pinref part="GND32" gate="1" pin="GND"/>
 <wire x1="76.2" y1="-116.84" x2="76.2" y2="-119.38" width="0.1524" layer="91"/>
@@
 </segment>
 <segment>
-<pinref part="GND3" gate="1" pin="GND"/>
-<pinref part="D1" gate="G$1" pin="A"/>
-<wire x1="-96.52" y1="114.3" x2="-96.52" y2="116.84" width="0.1524" layer="91"/>
-</segment>
-<segment>
-<pinref part="GND6" gate="1" pin="GND"/>
-<pinref part="D2" gate="G$1" pin="A"/>
-<wire x1="-96.52" y1="73.66" x2="-96.52" y2="76.2" width="0.1524" layer="91"/>
-</segment>
-<segment>
 <pinref part="R9" gate="G$1" pin="1"/>
 <pinref part="GND13" gate="1" pin="GND"/>
@@
 <pinref part="R6" gate="G$1" pin="1"/>
 <pinref part="GND23" gate="1" pin="GND"/>
+</segment>
+<segment>
+<pinref part="B1" gate="G$1" pin="-"/>
+<pinref part="GND28" gate="1" pin="GND"/>
+<wire x1="-119.38" y1="121.92" x2="-121.92" y2="121.92" width="0.1524" layer="91"/>
+<wire x1="-121.92" y1="121.92" x2="-121.92" y2="111.76" width="0.1524" layer="91"/>
+</segment>
+<segment>
+<pinref part="B2" gate="G$1" pin="-"/>
+<pinref part="GND5" gate="1" pin="GND"/>
+<wire x1="-119.38" y1="81.28" x2="-121.92" y2="81.28" width="0.1524" layer="91"/>
+<wire x1="-121.92" y1="81.28" x2="-121.92" y2="71.12" width="0.1524" layer="91"/>
 </segment>
 </net>
@@
 <wire x1="-60.96" y1="-7.62" x2="-50.8" y2="-7.62" width="0.1524" layer="91"/>
 <label x="-55.88" y="-7.62" size="1.778" layer="95"/>
-</segment>
-</net>
-<net name="N$5" class="0">
-<segment>
-<wire x1="-111.76" y1="81.28" x2="-109.22" y2="81.28" width="0.1524" layer="91"/>
-<pinref part="R3" gate="G$1" pin="1"/>
-<pinref part="X7" gate="-2" pin="KL"/>
 </segment>
 </net>
@@
 <pinref part="+3V18" gate="G$1" pin="+3V3"/>
 </segment>
-<segment>
-<pinref part="D1" gate="G$1" pin="C"/>
-<pinref part="+3V2" gate="G$1" pin="+3V3"/>
-<wire x1="-96.52" y1="127" x2="-96.52" y2="129.54" width="0.1524" layer="91"/>
-</segment>
-<segment>
-<pinref part="D2" gate="G$1" pin="C"/>
-<pinref part="+3V5" gate="G$1" pin="+3V3"/>
-<wire x1="-96.52" y1="86.36" x2="-96.52" y2="88.9" width="0.1524" layer="91"/>
-</segment>
 </net>
 <net name="N$10" class="0">
@@
 </segment>
 </net>
-<net name="N$14" class="0">
-<segment>
-<wire x1="-111.76" y1="121.92" x2="-109.22" y2="121.92" width="0.1524" layer="91"/>
-<pinref part="R2" gate="G$1" pin="1"/>
-<pinref part="X6" gate="-2" pin="KL"/>
-</segment>
-<segment>
-<wire x1="-106.68" y1="119.38" x2="-104.14" y2="119.38" width="0.1524" layer="91"/>
-</segment>
-</net>
 <net name="N$7" class="0">
 <segment>
@@
 <wire x1="-60.96" y1="25.4" x2="-35.56" y2="25.4" width="0.1524" layer="91"/>
 <wire x1="-35.56" y1="25.4" x2="-35.56" y2="81.28" width="0.1524" layer="91"/>
-<pinref part="D6" gate="G$1" pin="C"/>
 <wire x1="-35.56" y1="81.28" x2="-78.74" y2="81.28" width="0.1524" layer="91"/>
 <pinref part="R9" gate="G$1" pin="2"/>
+<pinref part="B2" gate="G$1" pin="+"/>
+<wire x1="-109.22" y1="81.28" x2="-78.74" y2="81.28" width="0.1524" layer="91"/>
 <junction x="-78.74" y="81.28"/>
-<wire x1="-78.74" y1="81.28" x2="-81.28" y2="81.28" width="0.1524" layer="91"/>
 </segment>
 </net>
@@
 <pinref part="IC1" gate="G$1" pin="PC0(ADC0)"/>
 <wire x1="-27.94" y1="43.18" x2="-60.96" y2="43.18" width="0.1524" layer="91"/>
-<pinref part="D5" gate="G$1" pin="C"/>
-<wire x1="-81.28" y1="121.92" x2="-78.74" y2="121.92" width="0.1524" layer="91"/>
 <pinref part="R6" gate="G$1" pin="2"/>
+<wire x1="-78.74" y1="121.92" x2="-27.94" y2="121.92" width="0.1524" layer="91"/>
+<pinref part="B1" gate="G$1" pin="+"/>
+<wire x1="-109.22" y1="121.92" x2="-78.74" y2="121.92" width="0.1524" layer="91"/>
 <junction x="-78.74" y="121.92"/>
-<wire x1="-78.74" y1="121.92" x2="-27.94" y2="121.92" width="0.1524" layer="91"/>
 </segment>
 </net>
@@
 </segment>
 </net>
+<net name="N$8" class="0">
+<segment>
+<pinref part="X6" gate="-1" pin="KL"/>
+<pinref part="B1" gate="G$1" pin="AC2"/>
+<wire x1="-127" y1="114.3" x2="-114.3" y2="114.3" width="0.1524" layer="91"/>
+<wire x1="-114.3" y1="114.3" x2="-114.3" y2="116.84" width="0.1524" layer="91"/>
+</segment>
+</net>
+<net name="N$13" class="0">
+<segment>
+<pinref part="X6" gate="-2" pin="KL"/>
+<pinref part="B1" gate="G$1" pin="AC1"/>
+<wire x1="-127" y1="129.54" x2="-114.3" y2="129.54" width="0.1524" layer="91"/>
+<wire x1="-114.3" y1="129.54" x2="-114.3" y2="127" width="0.1524" layer="91"/>
+</segment>
+</net>
 <net name="N$1" class="0">
 <segment>
-<pinref part="R2" gate="G$1" pin="2"/>
-<pinref part="D1" gate="G$1" pin="AC"/>
-<pinref part="D5" gate="G$1" pin="A"/>
-<wire x1="-99.06" y1="121.92" x2="-86.36" y2="121.92" width="0.1524" layer="91"/>
-</segment>
-</net>
-<net name="N$6" class="0">
-<segment>
-<pinref part="R3" gate="G$1" pin="2"/>
-<pinref part="D2" gate="G$1" pin="AC"/>
-<pinref part="D6" gate="G$1" pin="A"/>
-<wire x1="-86.36" y1="81.28" x2="-99.06" y2="81.28" width="0.1524" layer="91"/>
-</segment>
-</net>
+<pinref part="X7" gate="-2" pin="KL"/>
+<pinref part="B2" gate="G$1" pin="AC1"/>
+<wire x1="-127" y1="88.9" x2="-114.3" y2="88.9" width="0.1524" layer="91"/>
+<wire x1="-114.3" y1="88.9" x2="-114.3" y2="86.36" width="0.1524" layer="91"/>
+</segment>
+</net>
+<net name="N$5" class="0">
+<segment>
+<pinref part="X7" gate="-1" pin="KL"/>
+<pinref part="B2" gate="G$1" pin="AC2"/>
+<wire x1="-127" y1="73.66" x2="-114.3" y2="73.66" width="0.1524" layer="91"/>
+<wire x1="-114.3" y1="73.66" x2="-114.3" y2="76.2" width="0.1524" layer="91"/>
+</segment>
+</net>
